Commit message: Removed collision models to prevent errors for the moment. Alternative is to host them in this package.

File: descartes_benchmarks/config/ur5_demo.urdf (robot description, URDF)
Before this commit: robot ur5_demo, 10 links, 9 joints
Links:
- link base_link: geometry 
- link forearm_link: geometry 
- link shoulder_link: geometry 
- link tool: geometry collision box size=0.04 0.04 0.06; collision cylinder length=0.02 radius=0.02
- link upper_arm_link: geometry 
- link wrist_1_link: geometry 
- link wrist_2_link: geometry 
- link wrist_3_link: geometry 
